File: kicad/RetroWiFiModem.sch (KiCad schematic (older format))
At the start: 38 parts, among them CON1 BARREL_JACK, P1 CONN_02X05, U1 74HC245, U2 MAX3232, U3 74HC32, U4 LP2950ACZ-3.3, U5 WeMos_D1_mini

Commit message: Initial commit for the v2 hardware. * MAX3237 for full suite of RS-232 control signals * DFPlayer Mini for faux dialing and connection sounds * Gerbers suitable for JLCPCB included
Parts:
- removed H1, H2, H3, H4, H5, H6: MountingHole, MountingHole:MountingHole_3.2mm_M3, symbol Mechanical:MountingHole
- removed U1: 74HC245, Package_DIP:DIP-20_W7.62mm, symbol 74xx:74HC245
- removed U2: MAX3232, Package_DIP:DIP-16_W7.62mm, symbol Interface_UART:MAX232
- removed unit 5 of U3
- added D9: 1N4148, modules:D_DO-35_SOD27_P7.62mm_Horizontal, symbol Diode:1N4148
- added LS1: Speaker, modules:PinHeader_1x02_P2.54mm_Vertical, symbol Device:Speaker
- added R10: 10K, modules:R3, symbol RetroWiFiModem:R_US
- added U1: MAX3237CAI+, modules:SOIC-28W_7.5x17.9mm_Pitch1.27mm, symbol RetroWiFiModem:MAX3237CAI+
- added U2: 74HCT245, modules:SOIC-20W_7.5x12.8mm_P1.27mm, symbol RetroWiFiModem:74LS245A
- added U6: DFPlayer_Mini, modules:DFPlayerMini, symbol RetroWiFiModem:DFPlayer_Mini
- C1, C2, C3, C4, C5, C7, C8: footprint Capacitor_THT:C_Disc_D3.0mm_W2.0mm_P2.50mm -> modules:C_Disc_D3_P2.5; symbol Device:C_Small -> RetroWiFiModem:C_Small
- C6: footprint Capacitor_THT:C_Disc_D5.0mm_W2.5mm_P5.00mm -> modules:R3; symbol Device:C_Small -> RetroWiFiModem:C_Small
- CON1: footprint Connector_BarrelJack:BarrelJack_Horizontal -> modules:BARREL_JACK; symbol Connector:Barrel_Jack_Switch -> RetroWiFiModem:BARREL_JACK
- D1, D2, D3, D4, D5, D6, D7, D8: footprint LED_THT:LED_D3.0mm -> modules:LED-3MM; symbol Device:LED -> RetroWiFiModem:LED
- P1: footprint Connector_IDC:IDC-Header_2x05_P2.54mm_Vertical -> modules:IDC_Header_Straight_10pins; symbol Connector_Generic:Conn_02x05_Odd_Even -> RetroWiFiModem:CONN_02X05
- R1: renamed from R8; footprint Resistor_THT:R_Axial_DIN0204_L3.6mm_D1.6mm_P7.62mm_Horizontal -> modules:DIP-16_W7.62mm_LongPads; symbol Device:R -> RetroWiFiModem:R_Pack08_US_Split
- R1: renamed from R7; footprint Resistor_THT:R_Axial_DIN0204_L3.6mm_D1.6mm_P7.62mm_Horizontal -> modules:DIP-16_W7.62mm_LongPads; symbol Device:R -> RetroWiFiModem:R_Pack08_US_Split
- R1: renamed from R6; footprint Resistor_THT:R_Axial_DIN0204_L3.6mm_D1.6mm_P7.62mm_Horizontal -> modules:DIP-16_W7.62mm_LongPads; symbol Device:R -> RetroWiFiModem:R_Pack08_US_Split
- R1: renamed from R5; footprint Resistor_THT:R_Axial_DIN0204_L3.6mm_D1.6mm_P7.62mm_Horizontal -> modules:DIP-16_W7.62mm_LongPads; symbol Device:R -> RetroWiFiModem:R_Pack08_US_Split
- R1: renamed from R4; footprint Resistor_THT:R_Axial_DIN0204_L3.6mm_D1.6mm_P7.62mm_Horizontal -> modules:DIP-16_W7.62mm_LongPads; symbol Device:R -> RetroWiFiModem:R_Pack08_US_Split
- R1: renamed from R3; footprint Resistor_THT:R_Axial_DIN0204_L3.6mm_D1.6mm_P7.62mm_Horizontal -> modules:DIP-16_W7.62mm_LongPads; symbol Device:R -> RetroWiFiModem:R_Pack08_US_Split
- R1: renamed from R2; footprint Resistor_THT:R_Axial_DIN0204_L3.6mm_D1.6mm_P7.62mm_Horizontal -> modules:DIP-16_W7.62mm_LongPads; symbol Device:R -> RetroWiFiModem:R_Pack08_US_Split
- R1: footprint Resistor_THT:R_Axial_DIN0204_L3.6mm_D1.6mm_P7.62mm_Horizontal -> modules:DIP-16_W7.62mm_LongPads; symbol Device:R -> RetroWiFiModem:R_Pack08_US_Split
- R9: footprint Resistor_THT:R_Axial_DIN0204_L3.6mm_D1.6mm_P7.62mm_Horizontal -> modules:R3; symbol Device:R -> RetroWiFiModem:R_US
- U3: footprint Package_DIP:DIP-14_W7.62mm -> modules:SOIC-14_3.9x8.7mm_P1.27mm; symbol 74xx:74LS32 -> RetroWiFiModem:74LS32
- U4: value LP2950ACZ-3.3 -> L4931CZ33-AP; footprint Package_TO_SOT_THT:TO-92L_Inline_Wide -> modules:TO-92_Inline_Wide; symbol Regulator_Linear:LP2950-3.3_TO92 -> RetroWiFiModem:LM2931AZ-3.3_5.0
- U5: value WeMos_D1_mini -> WeMos_mini; footprint RetroWiFiModem-footprints:wemos-d1-mini -> modules:wemos-d1-mini-with-pin-header-and-connector; Price 7.24 -> (none)
Connections:
- net +3V3: now also C3.1, U3.14 (VCC), U3.14 (VCC), U3.14 (VCC), U3.14 (VCC), R10.1, U1.14 (SHDN), U1.26 (VCC)
- net +5V: now also U2.1 (A->B), U2.20 (VCC), U6.1 (VCC)
- net GND: now also U3.7 (GND), U3.7 (GND), U3.7 (GND), U3.7 (GND), U1.15 (MBAUD), U1.2 (GND), U2.10 (GND), U2.19 (CE), U6.10 (GND), U6.7 (GND); no longer C3.2
- net at U5.11 (D0): now also D9.2 (A), R10.2
- net at R9.2, U3.2, U5.12 (D5): now also U1.13 (EN)
- net at U5.13 (D6): now also U1.17 (T5IN), U2.6 (A4)
- net at U5.14 (D7): now also U1.20 (R2OUT), U2.9 (A7)
- net at U5.15 (D8): now also U1.23 (T2IN), U2.8 (A6)
- net at U5.3 (D4): now also U6.2 (RX)
- net at U5.4 (D3): now also U1.18 (R3OUT), U2.3 (A1)
- net at U5.5 (D2): now also U1.19 (T4IN), U2.2 (A0)
- net at U5.6 (D1): now also U1.22 (T3IN), U2.7 (A5)
- net at U5.7 (Rx): now also U1.21 (R1OUT), U2.4 (A2)
- net at C6.1: now also U1.28 (C1+)
- net at U3.3: now also U1.24 (T1IN), U2.5 (A3)
- net at P1.5 (P5): now also U1.8 (R1IN)
- net at P1.3 (P3): now also U1.5 (T1OUT)
- net at C2.1: now also U1.4 (V-)
- net at C6.2: now also U1.25 (C1-)
- net at C1.1: now also U1.1 (C2+)
- net at C1.2: now also U1.3 (C2-)
- net at P1.6 (P6): now also U1.6 (T2OUT)
- net at P1.4 (P4): now also U1.9 (R2IN)
- net at P1.1 (P1): now also U1.7 (T3OUT)
- net at P1.2 (P2): now also U1.10 (T4OUT)
- net at P1.7 (P7): now also U1.11 (R3IN)
- net at P1.8 (P8): now also U1.12 (T5OUT)
- net at D3.1 (K): now also R1.14 (R1.2); no longer R1.2
- net at D4.1 (K): now also R1.13 (R1.2); no longer R1.2
- net at D2.1 (K): now also R1.15 (R1.2); no longer R1.2
- net at D1.1 (K): now also R1.16 (R1.2); no longer R1.2
- net at D5.1 (K): now also R1.12 (R1.2); no longer R1.2
- net at D6.1 (K): now also R1.11 (R1.2); no longer R1.2
- net at D7.1 (K): now also R1.10 (R1.2); no longer R1.2
- net at D8.1 (K): now also R1.9 (R1.2); no longer R1.2
- net at R1.1 (R1.1): now also U2.18 (B0)
- new net: C3.2, U1.27 (V+)
- new net: R1.8 (R1.1), U2.11 (B7)
- new net: R1.7 (R1.1), U2.12 (B6)
- new net: R1.6 (R1.1), U2.13 (B5)
- new net: R1.5 (R1.1), U2.14 (B4)
- new net: R1.4 (R1.1), U2.15 (B3)
- new net: R1.3 (R1.1), U2.16 (B2)
- new net: R1.2 (R1.1), U2.17 (B1)
- new net: D9.1 (K), U6.16 (BUSY)
- new net: LS1.2, U6.6 (SPK+)
- new net: LS1.1, U6.8 (SPK-)
- no-connect marks 15 -> 18
Other:
- note added: "CD"
- note added: "CS"
- note added: "MR"
- note added: "RD"
- note added: "RS"
- note added: "SD"
- note added: "TR"
- note added: "TXEN"
- moved on the sheet: C2, C3, C5, C6, C8
